File: KiCad/Nostroino UNO.kicad_pcb (KiCad board)
At the start: 2 copper layers, 68.6 x 53.3 mm, 45 parts, among them J1 USB|EXT., U1 7805, U2 ATMEGA368P-PU, U3 FT232RL, X1 Alimentação, X10 Fix3, X11 Fix4, X2 USB, X3 POWER, X4 DIGITAL (PWM#)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

Commit message: Update Silk PCB
Parts:
- moved VAL 0.25 mm to (132.0, 104.9)
Other:
- board text added: "ARDUINO UNO - COMPATIBLE"
- board text added: "BOARD VERSION 2015.02.04"
- board text added: "Designed by"
- board text added: "NOSTROINO.GITHUB.IO"
- board text added: "TM"
- board text added: "creativecommons.org"
- board text removed: "Baseado em ARDUINO UNO R3"
- board text removed: "Desenvolvido por"
- board text removed: "creativecommons.org/licenses/by-sa/3.0/br"
- board text removed: "rev. 2015.01.20"
