File: KiCad/Nostroino UNO.kicad_pcb (KiCad board)
At the start: 2 copper layers, 68.6 x 53.3 mm, 45 parts, among them J1 USB|EXT., U1 7805, U2 ATMEGA368P-PU, U3 FT232RL, X1 Alimentação, X10 Fix3, X11 Fix4, X2 USB, X3 POWER, X4 DIGITAL (PWM#)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

Commit message: KiCad PCB Updat
- GND USB passando para trilha 1A;
- N-000004 passando para trilha 1A;
- Sinal “+” no footprint no Cap. 10uF;
- Aumentar furos do “EXT./USB” e ICSP;
- Atualização Board Version para 2015.02.05.
Routing:
- net GND: track 369.7 -> 390.3 mm
- net N-000004: track 14.4 -> 21.3 mm
Other:
- board text added: "+"
- board text added: "2015.02.05 11h02"
- board text added: "BOARD VERSION 2015.02.05"
- board text removed: "BOARD VERSION 2015.02.04"
Changed lines of the file:
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@@
     (links 99)
     (no_connects 0)
-    (area 79.679799 85.3948 154.990001 140.1572)
+    (area 79.679799 76.2224 154.990001 140.1572)
     (thickness 1.6)
-    (drawings 80)
-    (tracks 672)
+    (drawings 82)
+    (tracks 682)
     (zones 0)
     (modules 45)
@@
     (15 F.Cu signal)
     (0 B.Cu signal)
-    (16 B.Adhes user)
-    (17 F.Adhes user)
-    (18 B.Paste user)
-    (19 F.Paste user)
+    (16 B.Adhes user hide)
+    (17 F.Adhes user hide)
+    (18 B.Paste user hide)
+    (19 F.Paste user hide)
     (20 B.SilkS user)
     (21 F.SilkS user)
     (22 B.Mask user)
-    (23 F.Mask user)
-    (24 Dwgs.User user)
-    (25 Cmts.User user)
-    (26 Eco1.User user)
-    (27 Eco2.User user)
+    (23 F.Mask user hide)
+    (24 Dwgs.User user hide)
+    (25 Cmts.User user hide)
+    (26 Eco1.User user hide)
+    (27 Eco2.User user hide)
     (28 Edge.Cuts user)
   )
@@
     (mod_text_size 1 1)
     (mod_text_width 0.15)
-    (pad_size 5.08 5.08)
-    (pad_drill 2.794)
+    (pad_size 1.524 1.524)
+    (pad_drill 1.016)
     (pad_to_mask_clearance 0)
     (aux_axis_origin 0 0)
-    (visible_elements 7FFE7FFF)
+    (visible_elements 7FFEFFFF)
     (pcbplotparams
       (layerselection 1048576)
@@
     (add_net N-0000033)
     (add_net N-0000034)
-    (add_net N-000004)
     (add_net N-0000047)
     (add_net N-000005)
@@
     (add_net GND)
     (add_net N-000003)
+    (add_net N-000004)
     (add_net N-0000048)
     (add_net N-0000052)
@@
     (fp_line (start -0.635 1.27) (end -1.27 0.635) (layer F.SilkS) (width 0.1524))
     (fp_line (start -1.27 0.635) (end -1.27 -3.175) (layer F.SilkS) (width 0.1524))
-    (pad 6 thru_hole circle (at 5.08 -2.54 270) (size 1.524 1.524) (drill 0.889)
+    (pad 6 thru_hole circle (at 5.08 -2.54 270) (size 1.524 1.524) (drill 1.016)
       (layers *.Cu *.Mask)
       (net 13 GND)
     )
-    (pad 5 thru_hole circle (at 5.08 0 270) (size 1.524 1.524) (drill 0.889)
+    (pad 5 thru_hole circle (at 5.08 0 270) (size 1.524 1.524) (drill 1.016)
       (layers *.Cu *.Mask)
       (net 6 /RESET)
     )
-    (pad 3 thru_hole circle (at 2.54 0 270) (size 1.524 1.524) (drill 0.889)
+    (pad 3 thru_hole circle (at 2.54 0 270) (size 1.524 1.524) (drill 1.016)
       (layers *.Cu *.Mask)
       (net 8 /SCK)
     )
-    (pad 4 thru_hole circle (at 2.54 -2.54 270) (size 1.524 1.524) (drill 0.889)
+    (pad 4 thru_hole circle (at 2.54 -2.54 270) (size 1.524 1.524) (drill 1.016)
       (layers *.Cu *.Mask)
       (net 5 /MOSI)
     )
-    (pad 2 thru_hole circle (at 0 -2.54 270) (size 1.524 1.524) (drill 0.889)
+    (pad 2 thru_hole circle (at 0 -2.54 270) (size 1.524 1.524) (drill 1.016)
       (layers *.Cu *.Mask)
       (net 2 +5V)
     )
-    (pad 1 thru_hole circle (at 0 0 270) (size 1.524 1.524) (drill 0.889)
+    (pad 1 thru_hole circle (at 0 0 270) (size 1.524 1.524) (drill 1.016)
       (layers *.Cu *.Mask)
       (net 4 /MISO)
@@
     (fp_line (start 0.635 1.27) (end -0.635 1.27) (layer F.SilkS) (width 0.1524))
     (fp_line (start -0.635 1.27) (end -1.27 0.635) (layer F.SilkS) (width 0.1524))
-    (pad 3 thru_hole circle (at 5.08 0 90) (size 2.159 2.159) (drill 0.889)
+    (pad 3 thru_hole circle (at 5.08 0 90) (size 2.159 2.159) (drill 1.016)
       (layers *.Cu *.Mask)
       (net 33 N-000004)
     )
-    (pad 1 thru_hole circle (at 0 0 90) (size 2.159 2.159) (drill 0.889)
+    (pad 1 thru_hole circle (at 0 0 90) (size 2.159 2.159) (drill 1.016)
       (layers *.Cu *.Mask)
       (net 37 N-0000052)
     )
-    (pad 2 thru_hole circle (at 2.54 0 90) (size 2.159 2.159) (drill 0.889)
+    (pad 2 thru_hole circle (at 2.54 0 90) (size 2.159 2.159) (drill 1.016)
       (layers *.Cu *.Mask)
       (net 2 +5V)
@@
     )
   )
+  (gr_text "2015.02.05        11h02" (at 118.0465 77.851) (layer F.SilkS)
+    (effects (font (size 2 2) (thickness 0.1524)))
+  )
+  (gr_text + (at 104.14 130.048 90) (layer F.SilkS)
+    (effects (font (size 0.889 0.889) (thickness 0.1778)) (justify left))
+  )
   (gr_text TM (at 136.906 116.6495) (layer F.SilkS)
     (effects (font (size 0.55 0.6) (thickness 0.1143)) (justify left))
@@
     (effects (font (size 1.016 1.016) (thickness 0.1778)) (justify left mirror))
   )
-  (gr_text "BOARD VERSION 2015.02.04" (at 150.495 122.301) (layer B.SilkS)
+  (gr_text "BOARD VERSION 2015.02.05" (at 150.495 122.301) (layer B.SilkS)
     (effects (font (size 1.016 1.016) (thickness 0.1778)) (justify left mirror))
   )
@@
   (segment (start 142.494 114.935) (end 143.256 114.173) (width 0.3048) (layer F.Cu) (net 12))
   (segment (start 143.764 111.76) (end 146.05 111.76) (width 0.3048) (layer F.Cu) (net 12) (status 20))
+  (segment (start 92.075 102.87) (end 89.916 102.87) (width 1.016) (layer B.Cu) (net 13))
+  (segment (start 98.552 96.647) (end 98.552 92.964) (width 1.016) (layer B.Cu) (net 13))
+  (segment (start 96.9645 98.2345) (end 98.552 96.647) (width 1.016) (layer B.Cu) (net 13))
+  (segment (start 90.2335 98.2345) (end 96.9645 98.2345) (width 1.016) (layer B.Cu) (net 13))
+  (segment (start 88.7095 99.7585) (end 90.2335 98.2345) (width 1.016) (layer B.Cu) (net 13))
+  (segment (start 88.7095 101.6635) (end 88.7095 99.7585) (width 1.016) (layer B.Cu) (net 13))
+  (segment (start 89.916 102.87) (end 88.7095 101.6635) (width 1.016) (layer B.Cu) (net 13))
   (segment (start 92.075 131.445) (end 92.075 126.6825) (width 1.016) (layer F.Cu) (net 13))
   (segment (start 92.075 126.6825) (end 96.8375 121.92) (width 1.016) (layer F.Cu) (net 13))
@@
   (segment (start 112.776 90.90884) (end 112.776 88.9) (width 1.016) (layer B.Cu) (net 13))
   (segment (start 106.68 94.742) (end 106.68 94.234) (width 1.016) (layer B.Cu) (net 13))
-  (segment (start 106.68 94.234) (end 105.41 92.964) (width 1.016) (layer B.Cu) (net 13))
   (segment (start 105.41 92.964) (end 98.552 92.964) (width 1.016) (layer B.Cu) (net 13))
+  (segment (start 106.68 94.234) (end 105.41 92.964) (width 1.016) (layer B.Cu) (net 13))
   (segment (start 92.202 92.964) (end 98.552 92.964) (width 1.016) (layer B.Cu) (net 13))
   (segment (start 109.728 116.713) (end 108.331 116.713) (width 1.016) (layer B.Cu) (net 13))
@@
   (segment (start 153.289 114.3) (end 153.924 113.665) (width 0.3048) (layer F.Cu) (net 13))
   (segment (start 98.552 92.964) (end 105.664 92.964) (width 0.3048) (layer B.Cu) (net 13))
-  (segment (start 106.68 93.98) (end 106.045 93.345) (width 0.3048) (layer B.Cu) (net 13))
   (segment (start 105.664 92.964) (end 106.045 93.345) (width 0.3048) (layer B.Cu) (net 13))
+  (segment (start 106.68 93.98) (end 106.045 93.345) (width 0.3048) (layer B.Cu) (net 13))
   (segment (start 106.68 94.742) (end 106.68 93.98) (width 0.3048) (layer B.Cu) (net 13))
   (segment (start 110.617 93.345) (end 107.315 93.345) (width 0.3048) (layer B.Cu) (net 13))
@@
   (segment (start 118.11 105.41) (end 122.555 105.41) (width 0.3048) (layer F.Cu) (net 31) (status 20))
   (segment (start 118.11 101.6) (end 122.555 101.6) (width 0.3048) (layer F.Cu) (net 32) (status 20))
-  (segment (start 94.615 109.855) (end 93.345 108.585) (width 0.3048) (layer B.Cu) (net 33))
-  (segment (start 93.345 104.14) (end 94.615 102.87) (width 0.3048) (layer B.Cu) (net 33))
-  (segment (start 93.345 108.585) (end 93.345 104.14) (width 0.3048) (layer B.Cu) (net 33))
+  (segment (start 100.33 109.855) (end 94.615 109.855) (width 1.016) (layer B.Cu) (net 33))
+  (segment (start 94.615 102.87) (end 94.615 104.14) (width 1.016) (layer B.Cu) (net 33))
+  (segment (start 93.4085 109.855) (end 94.615 109.855) (width 1.016) (layer B.Cu) (net 33))
+  (segment (start 92.71 109.1565) (end 93.4085 109.855) (width 1.016) (layer B.Cu) (net 33))
+  (segment (start 92.71 106.045) (end 92.71 109.1565) (width 1.016) (layer B.Cu) (net 33))
+  (segment (start 94.615 104.14) (end 92.71 106.045) (width 1.016) (layer B.Cu) (net 33))
   (segment (start 100.965 109.855) (end 94.615 109.855) (width 0.3048) (layer B.Cu) (net 33) (status 30))
   (segment (start 127 119.38) (end 127 114.935) (width 0.3048) (layer B.Cu) (net 34) (status 30))

Commit message: KiCad
Adição de Zonas F. Cu e B. Cu
Routing:
- net GND: track 390.3 -> 388.0 mm
- net +3.3V: track 100.2 -> 99.5 mm
- added copper zone on B.Cu, net GND
- added copper zone on F.Cu, net GND
Other:
- board text added: "2015.02.05 15h23"
- board text removed: "2015.02.05 11h02"

Commit message: Update to KiCad 4.0.2
Routing:
- net GND: track 388.0 -> 369.7 mm
- net N-000004: track 21.3 -> 14.4 mm
- net +3.3V: track 99.5 -> 100.2 mm
- removed copper zone on B.Cu, net GND
- removed copper zone on F.Cu, net GND
Other:
- board text added: "BOARD VERSION 2015.02.04"
- board text added: "NOSTROINO.GITHUB.IO"
- board text removed: "+"
- board text removed: "2015.02.05 15h23"
- board text removed: "BOARD VERSION 2015.02.05"
- board text removed: "nostroino.github.io"
