File: KiCad/Nostroino UNO.sch (KiCad schematic (older format))
At the start: 38 parts, among them J1 USB/EXT, U1 7805, U2 ATMEGA368P-PU, U3 FT232RL, X1 Alimentação, X10 Fix3, X11 Fix4, X2 USB, X3 POWER, X4 DIGITAL (PWM#)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

Commit message: Update to KiCad 4.0.2
Parts:
- C1, C6, C7, C8, C9: footprint ~ -> Nostroino_UNO:Capacitor_100nFx63V; symbol CAPACITOR -> Capacitor
- C3, C4: footprint ~ -> Nostroino_UNO:Capacitor_15pF; symbol CAPACITOR -> Capacitor
- C5: footprint ~ -> Nostroino_UNO:Capacitor_10uFx50V_horizontal; symbol CAPACITOR_ELETROLITICO -> Capacitor_eletrolitico
- CH1: footprint ~ -> Nostroino_UNO:Chave_tactil_4_terminais_6x6mm; symbol CHAVE_TACTIL -> Chave_tactil
- D1: footprint ~ -> Nostroino_UNO:Diodo_1A; symbol DIODO -> Diodo
- D2, D3, D4, D5: footprint ~ -> Nostroino_UNO:LED3mm
- J1: footprint ~ -> Nostroino_UNO:Barra_pino_estampado_simples_180graus_3x; symbol JUMPER_3_PINOS -> Jumper_3_pinos
- R1, R2, R3, R4, R5, R6, R7, R8: footprint ~ -> Nostroino_UNO:Resistor_0,5W; symbol RESISTOR -> Resistor
- U1: footprint ~ -> Nostroino_UNO:TO-220_horizontal
- U2: footprint (none) -> Nostroino_UNO:CI28DIP300
- U3: footprint ~ -> Nostroino_UNO:CI28SSOP
- X1: footprint ~ -> Nostroino_UNO:Conector_entrada_para_fonte; symbol CONECTOR_2X -> Conector_2x
- X10, X11, X8, X9: footprint ~ -> Nostroino_UNO:Ilha_furo_120mils; symbol CONECTOR_1X -> Conector_1x
- X2: footprint ~ -> Nostroino_UNO:Conector_USB_tipo_B
- X3, X7: footprint ~ -> Nostroino_UNO:Conector_pino_estampado_simples_180graus_8x; symbol CONECTOR_8X -> Conector_8x
- X4: footprint ~ -> Nostroino_UNO:Conector_pino_estampado_simples_180graus_10x; symbol CONECTOR_10X -> Conector_10x
- X5: footprint ~ -> Nostroino_UNO:Barra_pino_estampado_duplo_180graus_3x; symbol CONECTOR_3X2 -> Conector_3x2
- X6: footprint ~ -> (none); symbol CONECTOR_6X -> Conector_6x
- XTAL1: footprint ~ -> Nostroino_UNO:Cristal; symbol CRISTAL -> Cristal
Other:
- moved on the sheet: D5, U2
